File: blahajpcb.kicad_pcb (KiCad board)
At the start: 2 copper layers, 238 x 83 mm, 19 parts

Commit message: Add files via upload
Parts:
- removed the G*** at (213.8, 111.2)
- removed the G*** at (84.0, 89.2)
- removed the G*** at (198.5, 113.0)
- removed the G*** at (129.6, 82.9)
- removed the G*** at (51.0, 76.0)
- removed the G*** at (172.5, 112.2)
- removed the G*** at (208.0, 106.5)
- removed the G*** at (131.2, 131.2)
- removed the G*** at (89.5, 88.0)
- added G***: LOGO, LOGO, F.Cu at (213.5, 110.2)
- added G***: LOGO, LOGO, F.Cu at (195.0, 112.8)
- added G***: LOGO, LOGO, F.Cu at (129.2, 136.2)
- added G***: LOGO, LOGO, F.Cu at (88.2, 87.8)
- added G***: LOGO, LOGO, F.Cu at (48.5, 76.5)
- added G***: LOGO, LOGO, F.Cu at (83.0, 90.2)
- added G***: LOGO, LOGO, F.Cu at (131.8, 130.5)
- added G***: LOGO, LOGO, F.Cu at (129.5, 82.0)
- added G***: LOGO, LOGO, F.Cu at (208.8, 106.5)
- added G***: LOGO, LOGO, F.Cu at (170.0, 111.0)
- moved G*** 1.20 mm to (250.2, 112.9)

Commit message: Add files via upload
Parts:
- moved G*** 9.00 mm to (242.8, 89.2)
- moved G*** 1.95 mm to (248.7, 111.6)
Routing:
- net (no net): vias 0 -> 1
Changed lines of the file:
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@@
 	(footprint "LOGO"
 		(layer "F.Cu")
-		(at 242.5 98.25 90)
+		(at 242.75 89.25 90)
 		(property "Reference" "G***"
 			(at 0 0 90)
@@
 	(footprint "LOGO"
 		(layer "F.Cu")
-		(at 250.191619 112.888583)
+		(at 248.691619 111.638583)
 		(property "Reference" "G***"
 			(at 0 0 0)
@@
 	)
 	(gr_text "fly1ngf1sh"
-		(at 241.25 71.25 270)
+		(at 241.75 71.5 270)
 		(layer "F.SilkS")
 		(effects
 			(font
-				(size 3 3)
-				(thickness 0.4)
+				(size 2 2)
+				(thickness 0.25)
 			)
 			(justify left bottom)
 		)
+	)
+	(via
+		(at 241.75 100)
+		(size 5)
+		(drill 4)
+		(layers "F.Cu" "B.Cu")
+		(net 0)
 	)
 	(segment

Commit message: Add files via upload
Parts:
- added BT2: Battery_Cell, Battery:BatteryHolder_Keystone_3034_1x20mm, B.Cu at (124.8, 131.8)
- added BT3: Battery_Cell, Battery:BatteryHolder_Keystone_3034_1x20mm, B.Cu at (167.0, 108.8)
- added D3: LED, LED_THT:LED_D5.0mm, F.Cu at (108.2, 102.5)
- added D4: LED, LED_THT:LED_D5.0mm, F.Cu at (126.2, 116.8)
- added D5: LED, LED_THT:LED_D5.0mm, F.Cu at (143.3, 103.0)
- added D6: LED, LED_THT:LED_D5.0mm, F.Cu at (137.3, 93.8)
- added R3: R, Resistor_THT:R_Axial_DIN0207_L6.3mm_D2.5mm_P7.62mm_Horizontal, B.Cu at (103.8, 101.2)
- added R4: R, Resistor_THT:R_Axial_DIN0207_L6.3mm_D2.5mm_P7.62mm_Horizontal, B.Cu at (98.5, 107.5)
- added R5: R, Resistor_THT:R_Axial_DIN0207_L6.3mm_D2.5mm_P7.62mm_Horizontal, B.Cu at (170.2, 128.8)
- added R6: R, Resistor_THT:R_Axial_DIN0207_L6.3mm_D2.5mm_P7.62mm_Horizontal, B.Cu at (174.0, 96.0)
- BT1, R1, R2: moved to B.Cu
- moved R1 44.0 mm to (104.7, 87.8)
- moved BT1 41.7 mm to (87.2, 90.0), turned to 180 degrees
- moved D1 19.9 mm to (126.2, 100.2), turned to -90 degrees
- moved R2 14.0 mm to (101.1, 93.8)
- moved D2 10.2 mm to (115.0, 93.8)
Routing:
- net Net-(BT3-+): track 0.00 -> 71.7 mm
- net Net-(BT2-+): track 0.00 -> 71.4 mm
- net Net-(D4-A): track 0.00 -> 46.0 mm
- net Net-(BT2--): track 0.00 -> 39.5 mm
- net Net-(BT1--): track 51.9 -> 14.0 mm
- net Net-(BT3--): track 0.00 -> 37.8 mm
- net Net-(D5-A): track 0.00 -> 35.7 mm
- net Net-(D6-A): track 0.00 -> 33.6 mm
- net Net-(D3-A): track 0.00 -> 16.0 mm
- net Net-(BT1-+): track 56.1 -> 44.7 mm
- net Net-(D1-A): track 15.3 -> 24.1 mm
- net Net-(D2-A): track 13.1 -> 9.76 mm
