File: blahajpcb.kicad_sch (KiCad schematic)
At the start: 6 parts

Commit message: Add files via upload
Parts:
- added BT3: Battery_Cell, Battery:BatteryHolder_Keystone_3034_1x20mm, symbol Device:Battery_Cell
- added D3, D4, D5, D6: LED, LED_THT:LED_D5.0mm, symbol Device:LED
- added R3, R4, R5, R6: R, Resistor_THT:R_Axial_DIN0207_L6.3mm_D2.5mm_P7.62mm_Horizontal, symbol Device:R
Connections:
- net at BT2.1 (+): now also R3.1, R4.1
- net at BT2.2 (-): now also D3.1 (K), D4.1 (K)
- new net: BT3.1 (+), R5.1, R6.1
- new net: BT3.2 (-), D5.1 (K), D6.1 (K)
- new net: D6.2 (A), R6.2
- new net: D4.2 (A), R4.2
- new net: D3.2 (A), R3.2
- new net: D5.2 (A), R5.2
Other:
- moved on the sheet: D2, R2
